File: Kicad files/A-Max.sch (KiCad schematic (older format))
At the start: 11 parts, among them J1 DB23F, J2 Conn_02x10_Odd_Even_MountingP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, J3 DB23M, J5 DB19M, U1 74LS139, U2 74LS393

Commit message: .
.
Parts:
- J1: symbol Connector:DB23_Female_MountingHoles -> A-Max-rescue:DB23_Female_MountingHoles-Connector
- J3: symbol Connector:DB23_Male_MountingHoles -> A-Max-rescue:DB23_Male_MountingHoles-Connector
Changed lines of the file:
@@
 $EndComp
 $Comp
-L Connector:DB23_Female_MountingHoles J1
+L A-Max-rescue:DB23_Female_MountingHoles-Connector J1
 U 1 1 608E5C01
 P 2150 4500
@@
 $EndComp
 $Comp
-L Connector:DB23_Male_MountingHoles J3
+L A-Max-rescue:DB23_Male_MountingHoles-Connector J3
 U 1 1 608ED48F
 P 9500 4350
