File: Rev.1/Kicad files/Amiga2MacFloppy.kicad_pcb (KiCad board)
At the start: 2 copper layers, 44 x 48 mm, 12 parts, among them J1 DB23F, J2 Conn_02x10_Odd_Even_MountingP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, J3 DB23M, U1 74LS139, U2 74LS393

Commit message: Update
Update to board to add dimension and export it into the doc.
Parts:
- removed REF**: OSHW-Logo2_7.3x6mm_SilkScreen, Symbol:OSHW-Logo2_7.3x6mm_SilkScreen
- added R460: R1, Resistor_THT:R_Axial_DIN0204_L3.6mm_D1.6mm_P7.62mm_Horizontal, F.Cu at (127.2, 123.7)
- moved D1 14.2 mm to (142.1, 123.9)
- moved D2 2.62 mm to (142.1, 119.9)
- moved C1 1.24 mm to (128.4, 118.8)
- moved C2 1.17 mm to (143.5, 116.3)
Connections:
- net +5V renamed PWM
- J1 pad 20: Net-(J1-Pad20) -> (no net)
- J2 pad 17: Net-(J2-Pad17) -> (no net)
- J2 pad 19: Net-(J2-Pad19) -> (no net)
- J2 pad 9: Net-(J2-Pad9) -> (no net)
- U1 pad 10: Net-(U1-Pad10) -> (no net)
- U1 pad 11: Net-(U1-Pad11) -> (no net)
- U1 pad 5: Net-(U1-Pad5) -> (no net)
- U1 pad 6: Net-(U1-Pad6) -> (no net)
- U1 pad 7: Net-(U1-Pad7) -> (no net)
- U1 pad 9: Net-(U1-Pad9) -> (no net)
- U2 pad 10: Net-(U2-Pad10) -> (no net)
- U2 pad 11: Net-(U2-Pad11) -> (no net)
- U2 pad 12: Net-(U2-Pad12) -> (no net)
- U2 pad 13: Net-(U2-Pad13) -> (no net)
- U2 pad 4: Net-(U2-Pad4) -> (no net)
- U2 pad 5: Net-(U2-Pad5) -> (no net)
- U2 pad 6: Net-(U2-Pad6) -> (no net)
- U2 pad 8: Net-(U2-Pad8) -> (no net)
- U2 pad 9: Net-(U2-Pad9) -> (no net)
Routing:
- net _SEL2: track 41.5 -> 74.5 mm, vias 1 -> 2
- net Net-(D1-Pad1): track 30.9 -> 19.8 mm
- net PH2: track 73.9 -> 81.8 mm
- net RD: track 33.4 -> 25.8 mm
- net GND: track 135.3 -> 142.9 mm
- net PH3: track 75.8 -> 69.7 mm
- net _DKWE: track 64.8 -> 70.7 mm
- net _SEL1: track 41.1 -> 37.0 mm, vias 1 -> 0
- net DIR: track 71.4 -> 67.3 mm, vias 0 -> 1
- net _SEL3: track 41.2 -> 44.7 mm
- net _MTRXD: track 55.6 -> 57.9 mm
- net _DKRD: track 44.8 -> 47.0 mm
- net _DRES: track 41.0 -> 42.6 mm
- net _RDY: track 43.0 -> 44.4 mm
- net PH0: track 68.1 -> 69.1 mm
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